File: eMMC-microSD.sch (KiCad schematic (older format))
At the start: 0 parts

Commit message: Add mousebites to first adapter
Parts:
- added H1, H2: MountingHole, ToolingHole:ToolingHole_JLCSMT, symbol Mechanical:MountingHole
Changed lines of the file:
@@
 F1 "eMMC-adapter.sch" 50
 $EndSheet
+$Comp
+L Mechanical:MountingHole H1
+U 1 1 5F4D9869
+P 2150 2400
+F 0 "H1" H 2250 2446 50  0000 L CNN
+F 1 "MountingHole" H 2250 2355 50  0000 L CNN
+F 2 "ToolingHole:ToolingHole_JLCSMT" H 2150 2400 50  0001 C CNN
+F 3 "~" H 2150 2400 50  0001 C CNN
+	1    2150 2400
+	1    0    0    -1
+$EndComp
+$Comp
+L Mechanical:MountingHole H2
+U 1 1 5F4D9A43
+P 8750 4250
+F 0 "H2" H 8850 4296 50  0000 L CNN
+F 1 "MountingHole" H 8850 4205 50  0000 L CNN
+F 2 "ToolingHole:ToolingHole_JLCSMT" H 8750 4250 50  0001 C CNN
+F 3 "~" H 8750 4250 50  0001 C CNN
+	1    8750 4250
+	1    0    0    -1
+$EndComp
 $EndSCHEMATC
